Commit message: add toggle for joint state broadcaster

File: melfa_mon_description/ros2_control/monitor.hardware.xacro (robot description, xacro)
@@ -1,5 +1,5 @@
 <?xml version="1.0"?>
 <robot xmlns:xacro="http://www.ros.org/wiki/xacro">
-    <xacro:macro name="monitor_hardware" params="name prefix robot_ip send_port recv_port packet_lost_log  controller_config controller_type">
+    <xacro:macro name="monitor_hardware" params="name prefix robot_ip send_port recv_port packet_lost_log  controller_config controller_type joint_broadcaster">
         <xacro:property name="ctrl_limits" value="${xacro.load_yaml(controller_config)['controller_limits']}"/>
         <xacro:property name="ctrl_mode" value="${xacro.load_yaml(controller_config)['control_mode_io']}"/>
@@ -13,4 +13,5 @@
                 <param name="recv_port">${recv_port}</param>
                 <param name="packet_lost_log">${packet_lost_log}</param>
+                <param name="joint_broadcaster">${joint_broadcaster}</param>
                  <!-- Controller Type R/Q/D -->
                 <param name="controller_type">${controller_type}</param>
@@ -32,44 +33,46 @@
                 <param name="io_control_mode">${ctrl_mode['io_mode']}</param>
             </hardware>
-            <joint name="${prefix}joint_1">
-                <state_interface name="position"/>
-                <state_interface name="velocity"/>
-                <state_interface name="effort"/>
-            </joint>
-            <joint name="${prefix}joint_2">
-                <state_interface name="position"/>
-                <state_interface name="velocity"/>
-                <state_interface name="effort"/>
-            </joint>
-            <joint name="${prefix}joint_3">
-                <state_interface name="position"/>
-                <state_interface name="velocity"/>
-                <state_interface name="effort"/>
-            </joint>
-            <joint name="${prefix}joint_4">
-                <state_interface name="position"/>
-                <state_interface name="velocity"/>
-                <state_interface name="effort"/>
-            </joint>
-            <joint name="${prefix}joint_5">
-                <state_interface name="position"/>
-                <state_interface name="velocity"/>
-                <state_interface name="effort"/>
-            </joint>
-            <joint name="${prefix}joint_6">
-                <state_interface name="position"/>
-                <state_interface name="velocity"/>
-                <state_interface name="effort"/>
-            </joint>
-            <joint name="${prefix}joint_7">
-                <state_interface name="position"/>
-                <state_interface name="velocity"/>
-                <state_interface name="effort"/>
-            </joint>
-            <joint name="${prefix}joint_8">
-                <state_interface name="position"/>
-                <state_interface name="velocity"/>
-                <state_interface name="effort"/>
-            </joint>
+            <xacro:if value="${joint_broadcaster}">
+                <joint name="${prefix}joint_1">
+                    <state_interface name="position"/>
+                    <state_interface name="velocity"/>
+                    <state_interface name="effort"/>
+                </joint>
+                <joint name="${prefix}joint_2">
+                    <state_interface name="position"/>
+                    <state_interface name="velocity"/>
+                    <state_interface name="effort"/>
+                </joint>
+                <joint name="${prefix}joint_3">
+                    <state_interface name="position"/>
+                    <state_interface name="velocity"/>
+                    <state_interface name="effort"/>
+                </joint>
+                <joint name="${prefix}joint_4">
+                    <state_interface name="position"/>
+                    <state_interface name="velocity"/>
+                    <state_interface name="effort"/>
+                </joint>
+                <joint name="${prefix}joint_5">
+                    <state_interface name="position"/>
+                    <state_interface name="velocity"/>
+                    <state_interface name="effort"/>
+                </joint>
+                <joint name="${prefix}joint_6">
+                    <state_interface name="position"/>
+                    <state_interface name="velocity"/>
+                    <state_interface name="effort"/>
+                </joint>
+                <joint name="${prefix}joint_7">
+                    <state_interface name="position"/>
+                    <state_interface name="velocity"/>
+                    <state_interface name="effort"/>
+                </joint>
+                <joint name="${prefix}joint_8">
+                    <state_interface name="position"/>
+                    <state_interface name="velocity"/>
+                    <state_interface name="effort"/>
+                </joint>
+            </xacro:if>
             <xacro:macro name="gpio_interface" params="interface_name add_state_interfaces add_command_interfaces">
             <gpio name="${interface_name}">
@@ -106,5 +109,20 @@
                 <command_interface name="ctrl_type"/>
             </gpio>
-            <sensor name="${prefix}fts_raw_sensor">
+            <sensor name="fts_curr_sensor">
+                <state_interface name="force.x"/>
+                <state_interface name="force.y"/>
+                <state_interface name="force.z"/>
+                <state_interface name="torque.x"/>
+                <state_interface name="torque.y"/>
+                <state_interface name="torque.z"/>
+                <param name="frame_id">tool_1</param>
+                <param name="fx_range">1000</param>
+                <param name="fy_range">1000</param>
+                <param name="fz_range">1000</param>
+                <param name="tx_range">30</param>
+                <param name="ty_range">30</param>
+                <param name="tz_range">30</param>
+            </sensor>
+            <sensor name="fts_before_offset_sensor">
                 <state_interface name="force.x"/>
                 <state_interface name="force.y"/>
@@ -121,5 +139,5 @@
                 <param name="tz_range">30</param>
             </sensor>
-            <sensor name="${prefix}fts_before_offset_sensor">
+            <sensor name="fts_after_offset_sensor">
                 <state_interface name="force.x"/>
                 <state_interface name="force.y"/>
@@ -128,20 +146,5 @@
                 <state_interface name="torque.y"/>
                 <state_interface name="torque.z"/>
-                <param name="frame_id">default_tcp</param>
-                <param name="fx_range">1000</param>
-                <param name="fy_range">1000</param>
-                <param name="fz_range">1000</param>
-                <param name="tx_range">30</param>
-                <param name="ty_range">30</param>
-                <param name="tz_range">30</param>
-            </sensor>
-            <sensor name="${prefix}fts_after_offset_sensor">
-                <state_interface name="force.x"/>
-                <state_interface name="force.y"/>
-                <state_interface name="force.z"/>
-                <state_interface name="torque.x"/>
-                <state_interface name="torque.y"/>
-                <state_interface name="torque.z"/>
-                <param name="frame_id">default_tcp</param>
+                <param name="frame_id">tool_1</param>
                 <param name="fx_range">1000</param>
                 <param name="fy_range">1000</param>

File: melfa_mon_description/urdf/monitor.urdf.xacro (robot description, xacro)
@@ -9,13 +9,7 @@
     <xacro:arg name="controller_config" default="custom_monitor_params.yaml" />
     <xacro:arg name="packet_lost_log" default="1" />
-    <!-- Import urdf file -->
-    <!-- <xacro:include filename="$(find melfa_mon_description)/urdf/rv7frl/rv7frl_macro.xacro" /> -->
+    <xacro:arg name="joint_broadcaster" default="true" />
     <!-- Import ros2_control description -->
     <xacro:include filename="$(find melfa_mon_description)/ros2_control/monitor.hardware.xacro" />
-    <!-- Use world link to fix robot -->
-    <!-- <link name="$(arg prefix)world"/>
-    <xacro:rv7frl parent="$(arg prefix)world" prefix="$(arg prefix)">
-        <origin xyz="0 0 0" rpy="0 0 0" />
-    </xacro:rv7frl> -->
     <xacro:monitor_hardware
         name="rc1"
@@ -27,4 +21,5 @@
         controller_type="$(arg controller_type)"
         packet_lost_log="$(arg packet_lost_log)"
+        joint_broadcaster="$(arg joint_broadcaster)"
         />
 </robot>

Commit message: add pose_broadcaster,  motor state broadaster and robot_model parameter.

File: melfa_mon_description/ros2_control/monitor.hardware.xacro (robot description, xacro)
@@ -1,5 +1,5 @@
 <?xml version="1.0"?>
 <robot xmlns:xacro="http://www.ros.org/wiki/xacro">
-    <xacro:macro name="monitor_hardware" params="name prefix robot_ip send_port recv_port packet_lost_log  controller_config controller_type joint_broadcaster">
+    <xacro:macro name="monitor_hardware" params="name robot_model robot_ip send_port recv_port packet_lost_log  controller_config controller_type joint_broadcaster">
         <xacro:property name="ctrl_limits" value="${xacro.load_yaml(controller_config)['controller_limits']}"/>
         <xacro:property name="ctrl_mode" value="${xacro.load_yaml(controller_config)['control_mode_io']}"/>
@@ -8,5 +8,5 @@
             <hardware>
                 <plugin>melfa_monitor/MELFAMonitorHardwareInterface</plugin>
-                <param name="prefix">${prefix}</param>
+                <param name="robot_model">${robot_model}</param>
                 <param name="robot_ip">${robot_ip}</param>
                 <param name="send_port">${send_port}</param>
@@ -34,43 +34,67 @@
             </hardware>
             <xacro:if value="${joint_broadcaster}">
-                <joint name="${prefix}joint_1">
+                <joint name="${robot_model}joint_1">
                     <state_interface name="position"/>
                     <state_interface name="velocity"/>
-                    <state_interface name="effort"/>
+                    <state_interface name="ampere_rms"/>
+                    <state_interface name="encoder_misscount"/>
+                    <state_interface name="encoder_temperature"/>
+                    <state_interface name="motor_voltage"/>
                 </joint>
-                <joint name="${prefix}joint_2">
+                <joint name="${robot_model}joint_2">
                     <state_interface name="position"/>
                     <state_interface name="velocity"/>
-                    <state_interface name="effort"/>
+                    <state_interface name="ampere_rms"/>
+                    <state_interface name="encoder_misscount"/>
+                    <state_interface name="encoder_temperature"/>
+                    <state_interface name="motor_voltage"/>
                 </joint>
-                <joint name="${prefix}joint_3">
+                <joint name="${robot_model}joint_3">
                     <state_interface name="position"/>
                     <state_interface name="velocity"/>
-                    <state_interface name="effort"/>
+                    <state_interface name="ampere_rms"/>
+                    <state_interface name="encoder_misscount"/>
+                    <state_interface name="encoder_temperature"/>
+                    <state_interface name="motor_voltage"/>
                 </joint>
-                <joint name="${prefix}joint_4">
+                <joint name="${robot_model}joint_4">
                     <state_interface name="position"/>
                     <state_interface name="velocity"/>
-                    <state_interface name="effort"/>
+                    <state_interface name="ampere_rms"/>
+                    <state_interface name="encoder_misscount"/>
+                    <state_interface name="encoder_temperature"/>
+                    <state_interface name="motor_voltage"/>
                 </joint>
-                <joint name="${prefix}joint_5">
+                <joint name="${robot_model}joint_5">
                     <state_interface name="position"/>
                     <state_interface name="velocity"/>
-                    <state_interface name="effort"/>
+                    <state_interface name="ampere_rms"/>
+                    <state_interface name="encoder_misscount"/>
+                    <state_interface name="encoder_temperature"/>
+                    <state_interface name="motor_voltage"/>
                 </joint>
-                <joint name="${prefix}joint_6">
+                <joint name="${robot_model}joint_6">
                     <state_interface name="position"/>
                     <state_interface name="velocity"/>
-                    <state_interface name="effort"/>
+                    <state_interface name="ampere_rms"/>
+                    <state_interface name="encoder_misscount"/>
+                    <state_interface name="encoder_temperature"/>
+                    <state_interface name="motor_voltage"/>
                 </joint>
-                <joint name="${prefix}joint_7">
+                <joint name="${robot_model}joint_7">
                     <state_interface name="position"/>
                     <state_interface name="velocity"/>
-                    <state_interface name="effort"/>
+                    <state_interface name="ampere_rms"/>
+                    <state_interface name="encoder_misscount"/>
+                    <state_interface name="encoder_temperature"/>
+                    <state_interface name="motor_voltage"/>
                 </joint>
-                <joint name="${prefix}joint_8">
+                <joint name="${robot_model}joint_8">
                     <state_interface name="position"/>
                     <state_interface name="velocity"/>
-                    <state_interface name="effort"/>
+                    <state_interface name="ampere_rms"/>
+                    <state_interface name="encoder_misscount"/>
+                    <state_interface name="encoder_temperature"/>
+                    <state_interface name="motor_voltage"/>
                 </joint>
             </xacro:if>
@@ -116,5 +140,5 @@
                 <state_interface name="torque.y"/>
                 <state_interface name="torque.z"/>
-                <param name="frame_id">tool_1</param>
+                <param name="frame_id">${robot_model}tool_0</param>
                 <param name="fx_range">1000</param>
                 <param name="fy_range">1000</param>
@@ -131,5 +155,5 @@
                 <state_interface name="torque.y"/>
                 <state_interface name="torque.z"/>
-                <param name="frame_id">default_tcp</param>
+                <param name="frame_id">${robot_model}default_tcp</param>
                 <param name="fx_range">1000</param>
                 <param name="fy_range">1000</param>
@@ -146,5 +170,5 @@
                 <state_interface name="torque.y"/>
                 <state_interface name="torque.z"/>
-                <param name="frame_id">tool_1</param>
+                <param name="frame_id">${robot_model}tool_1</param>
                 <param name="fx_range">1000</param>
                 <param name="fy_range">1000</param>
@@ -154,4 +178,14 @@
                 <param name="tz_range">30</param>
             </sensor>
+            <sensor name="${robot_model}tcp_pose">
+                <param name="frame_id">${robot_model}base</param>
+                <state_interface name="position.x"/>
+                <state_interface name="position.y"/>
+                <state_interface name="position.z"/>
+                <state_interface name="orientation.x"/>
+                <state_interface name="orientation.y"/>
+                <state_interface name="orientation.z"/>
+                <state_interface name="orientation.w"/>
+            </sensor>
         </ros2_control>
     </xacro:macro>

File: melfa_mon_description/urdf/monitor.urdf.xacro (robot description, xacro)
@@ -2,5 +2,5 @@
 <robot xmlns:xacro="http://www.ros.org/wiki/xacro" name="rc1">
     <!-- Enable setting arguments from the launch file -->
-    <xacro:arg name="prefix" default="" />
+    <xacro:arg name="robot_model" default="" />
     <xacro:arg name="robot_ip" default="192.168.0.20" />
     <xacro:arg name="send_port" default="12000" />
@@ -14,5 +14,5 @@
     <xacro:monitor_hardware
         name="rc1"
-        prefix="$(arg prefix)"
+        robot_model="$(arg robot_model)"
         robot_ip="$(arg robot_ip)"
         send_port="$(arg send_port)"

Commit message: add prefix and dynamic namespace function

File: melfa_mon_description/ros2_control/monitor.hardware.xacro (robot description, xacro)
@@ -1,5 +1,5 @@
 <?xml version="1.0"?>
 <robot xmlns:xacro="http://www.ros.org/wiki/xacro">
-    <xacro:macro name="monitor_hardware" params="name robot_model robot_ip send_port recv_port packet_lost_log  controller_config controller_type joint_broadcaster">
+    <xacro:macro name="monitor_hardware" params="name prefix robot_model robot_ip send_port recv_port packet_lost_log  controller_config controller_type joint_broadcaster">
         <xacro:property name="ctrl_limits" value="${xacro.load_yaml(controller_config)['controller_limits']}"/>
         <xacro:property name="ctrl_mode" value="${xacro.load_yaml(controller_config)['control_mode_io']}"/>
@@ -8,4 +8,5 @@
             <hardware>
                 <plugin>melfa_monitor/MELFAMonitorHardwareInterface</plugin>
+                <param name="prefix">${prefix}</param>
                 <param name="robot_model">${robot_model}</param>
                 <param name="robot_ip">${robot_ip}</param>
@@ -34,5 +35,5 @@
             </hardware>
             <xacro:if value="${joint_broadcaster}">
-                <joint name="${robot_model}joint_1">
+                <joint name="${prefix}${robot_model}${robot_model}joint_1">
                     <state_interface name="position"/>
                     <state_interface name="velocity"/>
@@ -42,5 +43,5 @@
                     <state_interface name="motor_voltage"/>
                 </joint>
-                <joint name="${robot_model}joint_2">
+                <joint name="${prefix}${robot_model}joint_2">
                     <state_interface name="position"/>
                     <state_interface name="velocity"/>
@@ -50,5 +51,5 @@
                     <state_interface name="motor_voltage"/>
                 </joint>
-                <joint name="${robot_model}joint_3">
+                <joint name="${prefix}${robot_model}joint_3">
                     <state_interface name="position"/>
                     <state_interface name="velocity"/>
@@ -58,5 +59,5 @@
                     <state_interface name="motor_voltage"/>
                 </joint>
-                <joint name="${robot_model}joint_4">
+                <joint name="${prefix}${robot_model}joint_4">
                     <state_interface name="position"/>
                     <state_interface name="velocity"/>
@@ -66,5 +67,5 @@
                     <state_interface name="motor_voltage"/>
                 </joint>
-                <joint name="${robot_model}joint_5">
+                <joint name="${prefix}${robot_model}joint_5">
                     <state_interface name="position"/>
                     <state_interface name="velocity"/>
@@ -74,5 +75,5 @@
                     <state_interface name="motor_voltage"/>
                 </joint>
-                <joint name="${robot_model}joint_6">
+                <joint name="${prefix}${robot_model}joint_6">
                     <state_interface name="position"/>
                     <state_interface name="velocity"/>
@@ -82,5 +83,5 @@
                     <state_interface name="motor_voltage"/>
                 </joint>
-                <joint name="${robot_model}joint_7">
+                <joint name="${prefix}${robot_model}joint_7">
                     <state_interface name="position"/>
                     <state_interface name="velocity"/>
@@ -90,5 +91,5 @@
                     <state_interface name="motor_voltage"/>
                 </joint>
-                <joint name="${robot_model}joint_8">
+                <joint name="${prefix}${robot_model}joint_8">
                     <state_interface name="position"/>
                     <state_interface name="velocity"/>
@@ -140,5 +141,5 @@
                 <state_interface name="torque.y"/>
                 <state_interface name="torque.z"/>
-                <param name="frame_id">${robot_model}tool_0</param>
+                <param name="frame_id">${prefix}${robot_model}tool_0</param>
                 <param name="fx_range">1000</param>
                 <param name="fy_range">1000</param>
@@ -155,5 +156,5 @@
                 <state_interface name="torque.y"/>
                 <state_interface name="torque.z"/>
-                <param name="frame_id">${robot_model}default_tcp</param>
+                <param name="frame_id">${prefix}${robot_model}default_tcp</param>
                 <param name="fx_range">1000</param>
                 <param name="fy_range">1000</param>
@@ -170,5 +171,5 @@
                 <state_interface name="torque.y"/>
                 <state_interface name="torque.z"/>
-                <param name="frame_id">${robot_model}tool_1</param>
+                <param name="frame_id">${prefix}${robot_model}tool_1</param>
                 <param name="fx_range">1000</param>
                 <param name="fy_range">1000</param>
@@ -178,6 +179,6 @@
                 <param name="tz_range">30</param>
             </sensor>
-            <sensor name="${robot_model}tcp_pose">
-                <param name="frame_id">${robot_model}base</param>
+            <sensor name="${prefix}${robot_model}tcp_pose">
+                <param name="frame_id">${prefix}${robot_model}base</param>
                 <state_interface name="position.x"/>
                 <state_interface name="position.y"/>

File: melfa_mon_description/urdf/monitor.urdf.xacro (robot description, xacro)
@@ -3,4 +3,5 @@
     <!-- Enable setting arguments from the launch file -->
     <xacro:arg name="robot_model" default="" />
+    <xacro:arg name="prefix" default="" />
     <xacro:arg name="robot_ip" default="192.168.0.20" />
     <xacro:arg name="send_port" default="12000" />
@@ -13,5 +14,6 @@
     <xacro:include filename="$(find melfa_mon_description)/ros2_control/monitor.hardware.xacro" />
     <xacro:monitor_hardware
-        name="rc1"
+        name="$(arg robot_model)"
+        prefix="$(arg prefix)"
         robot_model="$(arg robot_model)"
         robot_ip="$(arg robot_ip)"
