Commit message: scara compatibility

File: melfa_mon_description/ros2_control/monitor.hardware.xacro (robot description, xacro)
@@ -1,5 +1,5 @@
 <?xml version="1.0"?>
 <robot xmlns:xacro="http://www.ros.org/wiki/xacro">
-    <xacro:macro name="monitor_hardware" params="name prefix robot_model robot_ip send_port recv_port packet_lost_log  controller_config controller_type joint_broadcaster">
+    <xacro:macro name="monitor_hardware" params="name prefix robot_model robot_ip send_port recv_port packet_lost_log  controller_config controller_type joint_broadcaster scara">
         <xacro:property name="ctrl_limits" value="${xacro.load_yaml(controller_config)['controller_limits']}"/>
         <xacro:property name="ctrl_mode" value="${xacro.load_yaml(controller_config)['control_mode_io']}"/>
@@ -15,4 +15,5 @@
                 <param name="packet_lost_log">${packet_lost_log}</param>
                 <param name="joint_broadcaster">${joint_broadcaster}</param>
+                <param name="scara">${scara}</param>
                  <!-- Controller Type R/Q/D -->
                 <param name="controller_type">${controller_type}</param>
@@ -35,5 +36,5 @@
             </hardware>
             <xacro:if value="${joint_broadcaster}">
-                <joint name="${prefix}${robot_model}${robot_model}joint_1">
+                <joint name="${prefix}${robot_model}joint_1">
                     <state_interface name="position"/>
                     <state_interface name="velocity"/>

File: melfa_mon_description/urdf/monitor.urdf.xacro (robot description, xacro)
@@ -11,4 +11,5 @@
     <xacro:arg name="packet_lost_log" default="1" />
     <xacro:arg name="joint_broadcaster" default="true" />
+    <xacro:arg name="scara" default="0" />
     <!-- Import ros2_control description -->
     <xacro:include filename="$(find melfa_mon_description)/ros2_control/monitor.hardware.xacro" />
@@ -17,4 +18,5 @@
         prefix="$(arg prefix)"
         robot_model="$(arg robot_model)"
+        scara="$(arg scara)"
         robot_ip="$(arg robot_ip)"
         send_port="$(arg send_port)"
